File: hardware/project/ADC_Test/ADC.sch (KiCad schematic (older format))
At the start: 54 parts

Commit message: Development
Parts:
- removed C? (x13): 100n, Capacitor_SMD:C_0603_1608Metric_Pad1.05x0.95mm_HandSolder, symbol Device:C
- removed C?: 56p, symbol Device:C
- removed D? (x2): D, symbol Device:D_Capacitance
- removed R? (x2): 10k, symbol Device:R
- removed R? (x3): R, symbol Device:R
- removed R?: 82, symbol Device:R
- removed R? (x2): 51k, symbol Device:R
- removed R? (x2): 560, symbol Device:R
- removed U?: TL071, Package_SO:SOIC-8_3.9x4.9mm_P1.27mm, symbol Amplifier_Operational:TL071
- removed U? (x2): OPA140, Package_SO:SOIC-8_3.9x4.9mm_P1.27mm, symbol ADC_TEST:OPA140
- removed U?: OP07, symbol Amplifier_Operational:OP07
- removed U?: NE5534, symbol Amplifier_Operational:NE5534
- removed U?: LM311, symbol Comparator:LM311
- added C801: 33p, symbol Device:C
- added C802: DNP, symbol Device:C
- added C803: 100n, symbol Device:C
- added D801, D802, D803: BAV103, symbol Device:D
- added Q801: BC847W, Package_TO_SOT_SMD:SOT-323_SC-70, symbol Transistor_BJT:BC847W
- added R317: 1M, Resistor_SMD:R_0603_1608Metric_Pad1.05x0.95mm_HandSolder, symbol Device:R
- added R801, R803: 120k, symbol Device:R
- added R802: 620k, symbol Device:R
- added R804, R807: 12k, symbol Device:R
- added R805, R806, R809, R810, R813: 10, symbol Device:R
- added R808: 63k, symbol Device:R
- added R811: 620, symbol Device:R
- added R812, R816: 3k9, symbol Device:R
- added R814: 62, symbol Device:R
- added R815: 39k, symbol Device:R
- added TP801, TP802, TP803: TestPoint, symbol Connector:TestPoint
- added U801, U803: OPA177, symbol ADC_TEST:OPA177
- added U802: OPA140, symbol ADC_TEST:OPA140
- added U804: OPA192, symbol ADC_TEST:OPA192
- added U805: LM311, symbol Comparator:LM311
- C415: renamed from C?; value 2n2/THT -> 23PS222; footprint Capacitor_SMD:C_0603_1608Metric_Pad1.05x0.95mm_HandSolder -> Capacitor_THT:C_Axial_L12.0mm_D6.5mm_P15.00mm_Horizontal
- R404: renamed from R?; value 0 -> 62
- R406: renamed from R?; value 6k98/.05% -> 6k95/.05%
- R407, R408: renamed from R?; footprint Resistor_SMD:R_0805_2012Metric_Pad1.15x1.40mm_HandSolder -> Resistor_SMD:R_0603_1608Metric_Pad1.05x0.95mm_HandSolder
- U401: renamed from U?; footprint Package_SO:TSSOP-16_4.4x5mm_P0.65mm -> (none)
- U403: renamed from U?; value AD8676 -> OPA2192; symbol ADC_TEST:AD8676 -> ADC_TEST:OPA2192
- gave numbers to parts that had none: 8
Connections:
- net labels added: +18VF, +3.3VF, -14VF, -18VF, AD_COMP, DGNDF, FGPA_AD_ID, FGPA_AD_IIN, FGPA_AD_IRN, FGPA_AD_IRP, FPGA_AD_RFS, VR_-7V
- net labels removed: +10VREF, +15VF, +7VREF, -15VF, COMP, FGPA_SW_ID, FGPA_SW_IN, FGPA_SW_IR+, FGPA_SW_IR-
- wire segments 191 -> 212
- no-connect marks 10 -> 8
Other:
- moved on the sheet: C415, C416, C421, R404, R406, R407, R408, R410, U401A, U401B, U401C, U401D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
