File: hardware/project/ADC_Test/ADC_Test.sch (KiCad schematic (older format))
At the start: 1 part

Commit message: Development
Parts:
- added J102: Conn_01x02_Male, Connector_PinHeader_2.54mm:PinHeader_1x02_P2.54mm_Vertical, symbol Connector:Conn_01x02_Male
- added J103: Conn_01x04_Male, Connector_PinHeader_2.54mm:PinHeader_1x04_P2.54mm_Vertical, symbol Connector:Conn_01x04_Male
- J101: renamed from J?; footprint (none) -> ADC_TEST:36107406S
Connections:
- new net FPGA/FPGA_SPI3_MISO: J103.2 (Pin_2)
- new net FPGA/FPGA_SPI3_MOSI: J103.1 (Pin_1)
- new net FPGA/FPGA_SPI3_NSS: J103.4 (Pin_4)
- new net FPGA/FPGA_SPI3_SCK: J103.3 (Pin_3)
- new net FPGA/FPGA_UART2_RX_TTL: J102.1 (Pin_1)
- new net FPGA/FPGA_UART2_TX_TTL: J102.2 (Pin_2)
Other:
- moved on the sheet: J101
