File: hardware/project/ADC_Test/Connector.sch (KiCad schematic (older format))
At the start: 1 part

Commit message: Development
Parts:
- gave numbers to parts that had none: 1
Changed lines of the file:
@@
 $Descr A4 11693 8268
 encoding utf-8
-Sheet 6 7
+Sheet 3 8
 Title "Connector"
 Date "2020-03-07"
@@
 	5350 5050 5400 5050
 $Comp
-L power:Earth #PWR?
+L power:Earth #PWR0602
 U 1 1 5DECE77F
 P 5350 5050
-F 0 "#PWR?" H 5350 4800 50  0001 C CNN
+F 0 "#PWR0602" H 5350 4800 50  0001 C CNN
 F 1 "Earth" H 5350 4900 50  0001 C CNN
 F 2 "" H 5350 5050 50  0001 C CNN
@@
 	5450 7100 5400 7100
 $Comp
-L Connector:C64AC J?
+L Connector:C64AC J601
 U 1 1 5DE8758D
 P 5750 4000
-F 0 "J?" H 5930 4096 50  0000 L CNN
+F 0 "J601" H 5930 4096 50  0000 L CNN
 F 1 "C64AC" H 5930 4005 50  0000 L CNN
 F 2 "ADC_TEST:Socket_DIN41612-CaseC1-AC-Male-64Pin-2rows" H 5750 4050 50  0001 C CNN
@@
 $EndComp
 $Comp
-L ADC_TEST:+24VF #PWR?
+L ADC_TEST:+24VF #PWR0604
 U 1 1 60AC1A06
 P 5350 6950
-F 0 "#PWR?" H 5350 6800 50  0001 C CNN
+F 0 "#PWR0604" H 5350 6800 50  0001 C CNN
 F 1 "+24VF" V 5365 7077 50  0000 L CNN
 F 2 "" H 5350 6950 50  0001 C CNN
@@
 $EndComp
 $Comp
-L ADC_TEST:DGNDF #PWR?
+L ADC_TEST:DGNDF #PWR0603
 U 1 1 60AC7E80
 P 5350 6150
-F 0 "#PWR?" H 5350 5900 50  0001 C CNN
+F 0 "#PWR0603" H 5350 5900 50  0001 C CNN
 F 1 "DGNDF" V 5355 6023 50  0000 R CNN
 F 2 "" H 5350 6150 50  0001 C CNN
@@
 	5400 4300 5450 4300
 $Comp
-L power:Earth #PWR?
+L power:Earth #PWR0601
 U 1 1 5DED2C4C
 P 5350 4250
-F 0 "#PWR?" H 5350 4000 50  0001 C CNN
+F 0 "#PWR0601" H 5350 4000 50  0001 C CNN
 F 1 "Earth" H 5350 4100 50  0001 C CNN
 F 2 "" H 5350 4250 50  0001 C CNN
