File: hardware/project/ADC_Test/FPGA.sch (KiCad schematic (older format))
At the start: 72 parts

Commit message: Development
Parts:
- removed C? (x2): 100n, Capacitor_SMD:C_0603_1608Metric_Pad1.05x0.95mm_HandSolder, symbol Device:C
- removed R?: 150, Resistor_SMD:R_0603_1608Metric_Pad1.05x0.95mm_HandSolder, symbol Device:R
- removed U?: SN74LVC1T45DBV, Package_TO_SOT_SMD:SOT-23-6, symbol Logic_LevelTranslator:SN74LVC1T45DBV
- added Q701: BC857W, Package_TO_SOT_SMD:SOT-323_SC-70, symbol Transistor_BJT:BC857W
- added R722: 6k2, symbol Device:R
- gave numbers to parts that had none: 64
Connections:
- net SW_IN is gone; now on net SW_VRH: U505.4 (B)
- net SW_VRH: no longer R506.2, U501.4 (B)
- net at U503.37 (IOB_56): now also R722.2
- net FGPA_SW_ID renamed FGPA_AD_ID
- net FGPA_SW_IN renamed FGPA_SW_VRH
- net FGPA_SW_IR+ renamed FGPA_AD_IRP
- net FGPA_SW_IR- renamed FGPA_AD_IRN
- net FPGA_SPI1_MISO renamed FPGA_SPI3_MISO
- net FPGA_SPI1_MOSI renamed FPGA_SPI3_MOSI
- net FPGA_SPI1_NSS renamed FPGA_SPI3_NSS
- net FPGA_SPI1_SCK renamed FPGA_SPI3_SCK
- net FPGA_SW_VRH renamed FPGA_AD_IIN
- net FPGA_UART2_CTR_TTL renamed FPGA_UART2_CTRL_TTL
- net SW_ID renamed AD_ID
- net SW_IR+ renamed SW_IRP
- net SW_IR- renamed AD_IRN
- new net: Q701.1 (B), R722.1
- new net +3.3VF: Q701.2 (E)
- new net AD_IIN: U501.4 (B)
- new net FPGA_AD_RFS: Q701.3 (C)
Other:
- moved on the sheet: C501, C503, C505, C507, C512, C513, C514, C515, C516, C517, C518, C519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
