File: hardware/project/ADC_Test/MCU.sch (KiCad schematic (older format))
At the start: 36 parts

Commit message: Development
Parts:
- gave numbers to parts that had none: 36
Connections:
- net FPGA_SPI3_SCK: now reaches U201.111 (PC10,DFSDM1_CKIN5,SPI3_SCK,I2S3_CK,USART3_TX,UART4_TX,QUADSPI_BK1_IO1,SDMMC1_D2,DCMI_D8,LCD_R2,EVENTOUT)
- net FPGA_SPI3_MISO: now reaches U201.112 (PC11,DFSDM1_DATIN5,SPI3_MISO,USART3_RX,UART4_RX,QUADSPI_BK2_NCS,SDMMC1_D3,DCMI_D4,EVENTOUT)
- net FPGA_SPI3_MOSI: now reaches U201.113 (PC12,TRACED3,SPI3_MOSI,I2S3_SD,USART3_CK,UART5_TX,SDMMC1_CK,DCMI_D9,EVENTOUT)
- net MCU_ADC1_AZ: now reaches U201.56 (PG0,FMC_A10,EVENTOUT)
- net MCU_ADC2_AZ: now reaches U201.57 (PG1,FMC_A11,EVENTOUT)
- net AMPL_SEL: no longer names the net of U201.101 (PA9,TIM1_CH2,I2C3_SMBA,SPI2_SCK,I2S2_CK,USART1_TX,DCMI_D0,LCD_R5,EVENTOUT,OTG_FS_VBUS)
- net BA0 renamed RLY1_CTR
- net BA1: no longer names the net of U201.90 (PG5,FMC_A15,FMC_BA1,EVENTOUT)
- net CKE: no longer names the net of U201.135 (PB5,UART5_RX,TIM3_CH2,I2C1_SMBA,SPI1_MOSI,I2S1_SD,SPI3_MOSI,I2S3_SD,SPI6_MOSI,CAN2_RX,OTG_HS_ULPI_D7,ETH_PPS_OUT,FMC_SDCKE1,DCMI_D10,LCD_G7,EVENTOUT)
- net CLK: no longer names the net of U201.93 (PG8,SPI6_NSS,SPDIF_RX2,USART6_RTS,ETH_PPS_OUT,FMC_SDCLK,LCD_G7,EVENTOUT)
- net CXN_REL1: no longer names the net of U201.76 (PB15,RTC_REFIN,TIM1_CH3N,TIM8_CH3N,USART1_RX,SPI2_MOSI,I2S2_SD,DFSDM1_CKIN2,UART4_CTS,TIM12_CH2,SDMMC2_D1,OTG_HS_DP,EVENTOUT)
- net CXN_REL2 renamed AMP_10MEG
- net CXN_REL3 renamed RLY2_CTR
- net CXN_REL4: no longer names the net of U201.91 (PG6,FMC_NE3,DCMI_D12,LCD_R7,EVENTOUT)
- net CXN_REL5: no longer names the net of U201.92 (PG7,SAI1_MCLK_A,USART6_CK,FMC_INT,DCMI_D13,LCD_CLK,EVENTOUT)
- net DC_AMP2_MUX_A0: no longer names the net of U201.102 (PA10,TIM1_CH3,USART1_RX,LCD_B4,OTG_FS_ID,MDIOS_MDIO,DCMI_D1,LCD_B1,EVENTOUT)
- net DC_AMP2_MUX_A1: no longer names the net of U201.103 (PA11,TIM1_CH4,SPI2_NSS,I2S2_WS,UART4_RX,USART1_CTS,CAN1_RX,OTG_FS_DM,LCD_R4,EVENTOUT)
- net DC_AMP2_MUX_EN: no longer names the net of U201.104 (PA12,TIM1_ETR,SPI2_SCK,I2S2_CK,UART4_TX,USART1_RTS,SAI2_FS_B,CAN1_TX,OTG_FS_DP,LCD_R5,EVENTOUT)
- net DC_AMP_10MEG renamed FPGA_SPI3_NSS
- net FPGA_SPI1_MISO: no longer names the net of U201.124 (PG9,SPI1_MISO,SPDIF_RX3,USART6_RX,QUADSPI_BK2_IO2,SAI2_FS_B,SDMMC2_D0,FMC_NE2,FMC_NCE,DCMI_VSYNC,EVENTOUT)
- net FPGA_SPI1_MOSI renamed FPGA_UART2_CTRL_TTL
- net FPGA_SPI1_NSS: no longer names the net of U201.125 (PG10,SPI1_NSS,I2S1_WS,LCD_G3,SAI2_SD_B,SDMMC2_D1,FMC_NE3,DCMI_D2,LCD_B2,EVENTOUT)
- net FPGA_SPI1_SCK: no longer names the net of U201.41 (PA5,TIM2_CH1,TIM2_ETR,TIM8_CH1N,SPI1_SCK,I2S1_CK,SPI6_SCK,OTG_HS_ULPI_CK,LCD_R4,EVENTOUT,ADC1_IN5,ADC2_IN5,DAC_OUT2)
- net OCS_DIN: no longer names the net of U201.21 (PF9,SPI5_MOSI,SAI1_FS_B,UART7_CTS,TIM14_CH1,QUADSPI_BK1_IO1,EVENTOUT,ADC3_IN7)
- net OCS_SCLK: no longer names the net of U201.19 (PF7,TIM11_CH1,SPI5_SCK,SAI1_MCLK_B,UART7_TX,QUADSPI_BK1_IO2,EVENTOUT,ADC3_IN5)
- net OCS_SDO: no longer names the net of U201.20 (PF8,SPI5_MISO,SAI1_SCK_B,UART7_RTS,TIM13_CH1,QUADSPI_BK1_IO0,EVENTOUT,ADC3_IN6)
- net OCS_~SYNC: no longer names the net of U201.18 (PF6,TIM10_CH1,SPI5_NSS,SAI1_SD_B,UART7_RX,QUADSPI_BK1_IO3,EVENTOUT,ADC3_IN4)
- net ~CAS: no longer names the net of U201.132 (PG15,USART6_CTS,FMC_SDNCAS,DCMI_D13,EVENTOUT)
- net ~CS: no longer names the net of U201.136 (PB6,UART5_TX,TIM4_CH1,HDMI_CEC,I2C1_SCL,DFSDM1_DATIN5,USART1_TX,CAN2_TX,QUADSPI_BK1_NCS,I2C4_SCL,FMC_SDNE1,DCMI_D5,EVENTOUT)
- no-connect marks 72 -> 87
