File: hardware/project/ADC_Test/Power.sch (KiCad schematic (older format))
At the start: 70 parts, among them U401 TSR1-2490, U402 LM1117DTX-5.0/NOPB, U408 TSR1-2450, U409 LM1117DTX-3.3/NOPB

Commit message: Development
Parts:
- removed U?: MC7915BD2TG, Package_TO_SOT_SMD:TO-263-2, symbol Regulator_Linear:MC79M15_TO252
- removed U?: MC7815BD2TG, Package_TO_SOT_SMD:TO-263-2, symbol Regulator_Linear:L7815
- added C223: 10u/50V, Capacitor_SMD:C_1206_3216Metric_Pad1.42x1.75mm_HandSolder, symbol Device:C
- added C224, C228, C229, C230: 4u7/50V, Capacitor_SMD:C_1206_3216Metric_Pad1.42x1.75mm_HandSolder, symbol Device:C
- added C225: 1u, Capacitor_SMD:C_0603_1608Metric_Pad1.05x0.95mm_HandSolder, symbol Device:C
- added C226: 1u/HC, Capacitor_SMD:C_1206_3216Metric_Pad1.42x1.75mm_HandSolder, symbol Device:C
- added C227: 4p7, Capacitor_SMD:C_0603_1608Metric_Pad1.05x0.95mm_HandSolder, symbol Device:C
- added D204: PMEG6010EP,115, Diode_SMD:D_SOD-128, symbol Device:D_Schottky
- added L201: 74489440068, ADC_TEST:74489440068, symbol ADC_TEST:74489440068
- added R207, R208, R215: R, symbol Device:R
- added R209: 1k2, symbol Device:R
- added R210, R216: 120, symbol Device:R
- added R211, R213: 1M, Resistor_SMD:R_0603_1608Metric_Pad1.05x0.95mm_HandSolder, symbol Device:R
- added R212: 287k, Resistor_SMD:R_0603_1608Metric_Pad1.05x0.95mm_HandSolder, symbol Device:R
- added R214: 46k4, Resistor_SMD:R_0603_1608Metric_Pad1.05x0.95mm_HandSolder, symbol Device:R
- added U202: LM317_TO-263, Package_TO_SOT_SMD:TO-263-2, symbol Regulator_Linear:LM317_TO-263
- added U203, U205: LM337_TO263, Package_TO_SOT_SMD:TO-263-2, symbol Regulator_Linear:LM337_TO263
- added U204: LT8330_S6, Package_TO_SOT_SMD:TSOT-23-6_HandSoldering, symbol ADC_TEST:LT8330_S6
- gave numbers to parts that had none: 48
- renumbered C401 to C301, C402 to C302, C403 to C303, C409 to C309, C420 to C320, C425 to C325, C427 to C327, C431 to C331, C432 to C332, C434 to C334, C436 to C336, C437 to C337, L401 to L301, L404 to L304, U401 to U301, U402 to U302, U408 to U308, U409 to U309
Connections:
- net labels added: +18VF, -14VF, -18VF
- net labels removed: +15VF, -15VF
- wire segments 289 -> 363
Other:
- moved on the sheet: C304, C305, C307, C308, C310, C311, C312, C313, C316, C317, C318, C319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
